Commit message: python script

File: robotDescription/robot.urdf (robot description, URDF)
Before this commit: robot robotDescription, 1 links, 0 joints
Links:
- added link part_1_2, mass 5.0; collision mesh filename=package://assets/part_1__2.stl; visual mesh filename=package://assets/part_1__2.stl
- link part_1: mass 1e-09 -> 53.2845; geometry collision mesh filename=package://assets/part_1.stl; collision mesh filename=package://assets/part_1.stl
Joints:
- added joint slider_joint_part_1_2: type prismatic, parent part_1, child part_1_2, origin xyz=-0.015609 4.16334e-17 0.540048 rpy=-3.14159 0.523599 -3.14159, axis 1 0 0, limit lower=-0.5 upper=0.36 effort=100 velocity=10000.0

Commit message: mujoco description

File: robotDescription/robot.urdf (robot description, URDF)
Before this commit: robot robotDescription, 2 links, 1 joints
Joints:
- joint slider_joint_part_1_2: limit lower=-0.5 upper=0.36 effort=100 velocity=10000.0 -> lower=-0.36 upper=0.375 effort=100 velocity=10000.0
